Commit message: add gazebo sim

File: config/ros2_control.xacro (robot description, xacro)
@@ -89,4 +89,39 @@
         <state_interface name="velocity"/>
       </joint>
+      <!-- WHEEL JOINTS (Simulation only - hardware uses robot_controller.cpp) -->
+      <!-- Differential drive base with 4 wheels -->
+      <!-- Max velocity ±5.0 rad/s = ±0.15 m/s at wheel (0.03m radius) -->
+      <joint name="front_left_wheel_joint">
+        <command_interface name="velocity">
+          <param name="min">-5.0</param>
+          <param name="max">5.0</param>
+        </command_interface>
+        <state_interface name="position"/>
+        <state_interface name="velocity"/>
+      </joint>
+      <joint name="front_right_wheel_joint">
+        <command_interface name="velocity">
+          <param name="min">-5.0</param>
+          <param name="max">5.0</param>
+        </command_interface>
+        <state_interface name="position"/>
+        <state_interface name="velocity"/>
+      </joint>
+      <joint name="rear_left_wheel_joint">
+        <command_interface name="velocity">
+          <param name="min">-5.0</param>
+          <param name="max">5.0</param>
+        </command_interface>
+        <state_interface name="position"/>
+        <state_interface name="velocity"/>
+      </joint>
+      <joint name="rear_right_wheel_joint">
+        <command_interface name="velocity">
+          <param name="min">-5.0</param>
+          <param name="max">5.0</param>
+        </command_interface>
+        <state_interface name="position"/>
+        <state_interface name="velocity"/>
+      </joint>
     </ros2_control>
     <!-- Gazebo ros2_control plugin -->
