Commit message: fix(moveit): add mock_components hardware branch + fix gripper mimic
- ros2_control.xacro: add a `hardware` arg (mock|serial) with a
  mock_components/GenericSystem branch (default when not use_sim). Previously
  use_sim=false fell straight through to the unimplemented JetankSerialHardware
  plugin, so the controller manager could not load without Gazebo or motors.
- ros2_control.xacro: remove the gripper_right_joint <joint> block. It is a
  <mimic> of gripper_left_joint in the URDF; ros2_control forbids command
  interfaces on mimic joints and the mock/Ignition systems mirror it
  automatically.
- jetank_controllers.yaml: drop gripper_right_joint from gripper_controller
  joints (mimic, no command interface).

Verified: mock hardware loads and activates; joint_state_broadcaster
activates. Known open issue: arm_controller / gripper_controller do not yet
ingest their joints/command_interfaces params at configure time on
controller_manager 2.54 (RoboStack) — under investigation.

Part of feature/moveit-mock-arm.

Co-Authored-By: Claude Opus 4.8 (1M context) <noreply@anthropic.com>

File: config/ros2_control.xacro (robot description, xacro)
@@ -11,7 +11,12 @@
        Note: Exact mapping depends on hardware configuration
   -->
-  <xacro:macro name="jetank_ros2_control" params="use_sim:=true">
+  <!-- hardware: mock | serial  (only consulted when use_sim is false)
+       use_sim=true always selects the Gazebo/Ignition plugin. -->
+  <xacro:macro name="jetank_ros2_control" params="use_sim:=true hardware:='mock'">
     <ros2_control name="JetankSystem" type="system">
-      <!-- Hardware selection based on simulation flag -->
+      <!-- Hardware selection:
+           use_sim=true            -> Gazebo (Ignition) system
+           use_sim=false, serial   -> real Waveshare serial-bus servos
+           use_sim=false, mock     -> mock_components (software-only, no HW) -->
       <xacro:if value="${use_sim}">
         <hardware>
@@ -20,9 +25,16 @@
       </xacro:if>
       <xacro:unless value="${use_sim}">
-        <hardware>
-          <plugin>jetank_motor_control/JetankSerialHardware</plugin>
-          <param name="serial_port">/dev/ttyTHS1</param>
-          <param name="baud_rate">1000000</param>
-        </hardware>
+        <xacro:if value="${hardware == 'serial'}">
+          <hardware>
+            <plugin>jetank_motor_control/JetankSerialHardware</plugin>
+            <param name="serial_port">/dev/ttyTHS1</param>
+            <param name="baud_rate">1000000</param>
+          </hardware>
+        </xacro:if>
+        <xacro:unless value="${hardware == 'serial'}">
+          <hardware>
+            <plugin>mock_components/GenericSystem</plugin>
+          </hardware>
+        </xacro:unless>
       </xacro:unless>
       <!-- ARM JOINTS (S1-S5) -->
@@ -86,13 +98,8 @@
         <param name="servo_id">4</param>
       </joint>
-      <!-- gripper_right_joint is mimic of left in URDF, no direct control -->
-      <joint name="gripper_right_joint">
-        <command_interface name="position">
-          <param name="min">0.0</param>
-          <param name="max">0.04</param>
-        </command_interface>
-        <state_interface name="position"/>
-        <state_interface name="velocity"/>
-      </joint>
+      <!-- gripper_right_joint is a <mimic> of gripper_left_joint in the URDF.
+           ros2_control forbids command interfaces on mimic joints; both the
+           mock and Ignition systems mirror it automatically from the URDF
+           mimic tag, so it is intentionally NOT declared here. -->
       <!-- WHEEL JOINTS (Simulation only - hardware uses robot_controller.cpp) -->
       <!-- Differential drive base with 4 wheels -->

Commit message: docs(ros2_control): correct gripper mimic comment to match sim reality
Prior comment claimed Fortress enforces the URDF mimic in physics; Phase A
testing disproved this (left finger does not actuate in sim). Comment now
states the truth: control path is wired, real HW works via mechanical linkage,
but Fortress does not reliably enforce <mimic> — known sim limitation.

Co-Authored-By: Claude Opus 4.8 (1M context) <noreply@anthropic.com>

File: config/ros2_control.xacro (robot description, xacro)
@@ -79,10 +79,14 @@
            directly (JointGroupPositionController, one joint).
            gripper_right_joint is a URDF mimic of gripper_left_joint
-           (multiplier=1.0) — Gazebo Fortress enforces the mimic constraint
-           in physics, so the right finger follows the left automatically.
-           Giving gripper_right_joint a command_interface would create a
-           conflict between the controller setpoint and the physics mimic,
-           preventing the left finger from moving.  State interfaces remain
-           so joint_state_broadcaster can still publish both positions. -->
+           (multiplier=1.0), state-only here (no command interface).
+           REAL HARDWARE: one servo drives a mechanically-linked parallel jaw,
+           so commanding the single left joint is correct — the linkage moves
+           both fingers physically.
+           SIM CAVEAT (Gazebo Fortress / ign_ros2_control): the URDF <mimic>
+           tag is NOT reliably enforced in Fortress physics. The control path
+           is wired correctly (controller active, command accepted, state
+           published) but the left finger may not visibly actuate in sim.
+           Known limitation — tracked in the Phase A notes; arm motion (the
+           Phase A core goal) is fully functional. -->
       <joint name="gripper_left_joint">
         <command_interface name="position">

Commit message: fix(gripper): switch to GripperActionController + ros2_control native mimic
ros2_control.xacro:
- Add native mimic params to gripper_right_joint:
    <param name="mimic">gripper_left_joint</param>
    <param name="multiplier">1.0</param>
  ign_ros2_control parses these and mirrors the right finger without needing
  a Gazebo physics mimic constraint. The URDF <mimic> tag has been removed
  from gripper.xacro to eliminate the competing constraint.

jetank_controllers.yaml:
- Switch gripper_controller type from
    position_controllers/JointGroupPositionController
  to
    position_controllers/GripperActionController
  This exposes /gripper_controller/gripper_cmd (control_msgs/action/GripperCommand)
  instead of publishing Float64MultiArray on /gripper_controller/commands.
- Add GripperActionController params: joint, max_effort, allow_stalling,
  stall_velocity_threshold (0.0001), stall_timeout (10s), goal_tolerance.

Verified: position_controllers/GripperActionController active in Fortress;
gripper_left_joint moves to 0.04 m (open) and back to ~0.0 m (closed).

Co-Authored-By: Claude Opus 4.8 (1M context) <noreply@anthropic.com>

File: config/ros2_control.xacro (robot description, xacro)
@@ -76,17 +76,15 @@
       </joint>
       <!-- GRIPPER JOINTS -->
-      <!-- Gripper controlled by Servo 4: only the left finger is commanded
-           directly (JointGroupPositionController, one joint).
-           gripper_right_joint is a URDF mimic of gripper_left_joint
-           (multiplier=1.0), state-only here (no command interface).
-           REAL HARDWARE: one servo drives a mechanically-linked parallel jaw,
-           so commanding the single left joint is correct — the linkage moves
-           both fingers physically.
-           SIM CAVEAT (Gazebo Fortress / ign_ros2_control): the URDF <mimic>
-           tag is NOT reliably enforced in Fortress physics. The control path
-           is wired correctly (controller active, command accepted, state
-           published) but the left finger may not visibly actuate in sim.
-           Known limitation — tracked in the Phase A notes; arm motion (the
-           Phase A core goal) is fully functional. -->
+      <!-- gripper_left_joint is the COMMANDED joint (GripperActionController).
+           gripper_right_joint is mimic-only — no command interface.
+           The ros2_control resource manager's native mimic mechanism is used
+           (param name="mimic" + param name="multiplier") so that Gazebo
+           Fortress's ign_ros2_control properly mirrors the right finger to the
+           left.  The URDF <mimic> tag alone is NOT reliably enforced by Fortress
+           physics; the ros2_control params are the documented gz_ros2_control
+           pattern and work with GripperActionController.
+           REAL HARDWARE: one servo (ID 4) drives a mechanically-linked parallel
+           jaw, so commanding gripper_left_joint is correct — the linkage moves
+           both fingers physically. -->
       <joint name="gripper_left_joint">
         <command_interface name="position">
@@ -98,8 +96,11 @@
         <param name="servo_id">4</param>
       </joint>
-      <!-- gripper_right_joint: mimic joint — state only, no command interface. -->
+      <!-- gripper_right_joint: mimic joint — state only, no command interface.
+           ros2_control native mimic: resource manager mirrors left -> right. -->
       <joint name="gripper_right_joint">
         <state_interface name="position"/>
         <state_interface name="velocity"/>
+        <param name="mimic">gripper_left_joint</param>
+        <param name="multiplier">1.0</param>
       </joint>
       <!-- WHEEL JOINTS (Simulation only - hardware uses robot_controller.cpp) -->

Commit message: fix(gripper): replace ros2_control native mimic with separate command interface
Root cause of 'gripper_right_joint_mimic not found' spam and missing
right-finger TF: ign_ros2_control appends '_mimic' to the state
interface name when <param name="mimic"> is set, so joint_state_broadcaster
published 'gripper_right_joint_mimic' instead of 'gripper_right_joint'.

Changes:
- Remove <param name="mimic">/<param name="multiplier"> from
  gripper_right_joint in ros2_control.xacro. This eliminates the '_mimic'
  suffix; JSB now publishes 'gripper_right_joint' (the real URDF name).
- Give gripper_right_joint its own position command interface so Gazebo
  can physically move the right finger.
- Add gripper_right_mimic_controller (ForwardCommandController) to
  jetank_controllers.yaml, driven by the gripper_mimic_relay node.

Co-Authored-By: Claude Opus 4.8 (1M context) <noreply@anthropic.com>

File: config/ros2_control.xacro (robot description, xacro)
@@ -76,15 +76,25 @@
       </joint>
       <!-- GRIPPER JOINTS -->
-      <!-- gripper_left_joint is the COMMANDED joint (GripperActionController).
-           gripper_right_joint is mimic-only — no command interface.
-           The ros2_control resource manager's native mimic mechanism is used
-           (param name="mimic" + param name="multiplier") so that Gazebo
-           Fortress's ign_ros2_control properly mirrors the right finger to the
-           left.  The URDF <mimic> tag alone is NOT reliably enforced by Fortress
-           physics; the ros2_control params are the documented gz_ros2_control
-           pattern and work with GripperActionController.
-           REAL HARDWARE: one servo (ID 4) drives a mechanically-linked parallel
-           jaw, so commanding gripper_left_joint is correct — the linkage moves
-           both fingers physically. -->
+      <!-- gripper_left_joint: commanded by GripperActionController.
+           gripper_right_joint: has its OWN command interface (position) so Gazebo
+           enforces physical motion of the right finger independently.  A small
+           "gripper mimic relay" node (gripper_mimic_relay in
+           jetank_motor_control) subscribes to /joint_states and forwards the
+           gripper_left_joint position to the gripper_right_mimic_controller
+           (ForwardCommandController).  This makes BOTH fingers move in physics
+           and appear correctly in /joint_states.
+           The URDF <mimic> tag (restored in gripper.xacro) is kept for:
+             - robot_state_publisher TF computation when the relay is absent
+             - MoveIt joint model correctness
+             - RViz rendering fallback
+           The ros2_control NATIVE mimic params (<param name="mimic">/
+           <param name="multiplier">) are intentionally OMITTED because the gz
+           hardware plugin appends "_mimic" to the published state interface name,
+           producing "gripper_right_joint_mimic" in /joint_states — killing the
+           MoveIt joint-not-found spam required removing them.
+           REAL HARDWARE: one servo (ID 4) drives a mechanically-linked jaw; only
+           gripper_left_joint is commanding the servo; gripper_right_joint on
+           real hw has no servo and should not issue a command. The relay node
+           guards against this via use_sim_time check or a launch-time arg. -->
       <joint name="gripper_left_joint">
         <command_interface name="position">
@@ -96,11 +106,14 @@
         <param name="servo_id">4</param>
       </joint>
-      <!-- gripper_right_joint: mimic joint — state only, no command interface.
-           ros2_control native mimic: resource manager mirrors left -> right. -->
+      <!-- gripper_right_joint: own command interface so Gazebo can physically
+           move the right finger (driven by the mimic relay node). No native
+           ros2_control mimic params — avoids the _mimic suffix in JSB output. -->
       <joint name="gripper_right_joint">
+        <command_interface name="position">
+          <param name="min">0.0</param>
+          <param name="max">0.04</param>
+        </command_interface>
         <state_interface name="position"/>
         <state_interface name="velocity"/>
-        <param name="mimic">gripper_left_joint</param>
-        <param name="multiplier">1.0</param>
       </joint>
       <!-- WHEEL JOINTS (Simulation only - hardware uses robot_controller.cpp) -->

Commit message: Add JetankSerialHardware ros2_control driver, safe hardware mode, open-loop odom
- Implement JetankSerialHardware SystemInterface (src/hardware/) over a minimal
  Feetech SMS/STS serial protocol (feetech_bus, POSIX termios, no SDK dep).
  Joints with a servo_id do real I/O; others (gripper_right, wheels) mirror
  command->state. Per-joint offset/direction/ticks_per_rad calibration params.
- Wire the plugin into CMake (pluginlib export, shared lib jetank_serial_hardware)
  and fix jetank_hardware.xml library path; was a documented stub before.
- config/ros2_control.xacro: add 3-way hardware backend (sim|mock|serial) with a
  mock_components/GenericSystem branch. Closes the hazard where hardware:=mock
  silently selected the real serial plugin (drove real motors).
- robot_controller.cpp: publish open-loop odometry (/odom + odom->base_footprint)
  integrated from commanded velocity (drifts; no encoders). Adds nav_msgs/tf2 deps.

Compile-verified (build + uncrustify/cppcheck). NOT hardware-verified: the Feetech
register map/endianness is assumed and must be confirmed on real servos.

Co-Authored-By: Claude Opus 4.8 <noreply@anthropic.com>
Claude-Session: https://claude.ai/code/session_01DsqCvi8itGazj76ofFqPc7

File: config/ros2_control.xacro (robot description, xacro)
@@ -11,7 +11,14 @@
        Note: Exact mapping depends on hardware configuration
   -->
-  <xacro:macro name="jetank_ros2_control" params="use_sim:=true">
+  <xacro:macro name="jetank_ros2_control" params="use_sim:=true hardware:=mock">
     <ros2_control name="JetankSystem" type="system">
-      <!-- Hardware selection based on simulation flag -->
+      <!-- Hardware backend selection (3-way):
+             use_sim:=true            -> Gazebo IgnitionSystem (sim)
+             use_sim:=false hardware=mock   -> mock_components/GenericSystem
+                                               (software-only, NO motors move)
+             use_sim:=false hardware=serial -> JetankSerialHardware (real servos)
+           The mock branch is what makes `hardware:=mock` SAFE: previously the
+           xacro only knew use_sim, so a non-sim build always emitted the serial
+           plugin and `hardware:=mock` silently drove real motors. -->
       <xacro:if value="${use_sim}">
         <hardware>
@@ -20,9 +27,16 @@
       </xacro:if>
       <xacro:unless value="${use_sim}">
-        <hardware>
-          <plugin>jetank_motor_control/JetankSerialHardware</plugin>
-          <param name="serial_port">/dev/ttyTHS1</param>
-          <param name="baud_rate">1000000</param>
-        </hardware>
+        <xacro:if value="${hardware == 'mock'}">
+          <hardware>
+            <plugin>mock_components/GenericSystem</plugin>
+          </hardware>
+        </xacro:if>
+        <xacro:unless value="${hardware == 'mock'}">
+          <hardware>
+            <plugin>jetank_motor_control/JetankSerialHardware</plugin>
+            <param name="serial_port">/dev/ttyTHS1</param>
+            <param name="baud_rate">1000000</param>
+          </hardware>
+        </xacro:unless>
       </xacro:unless>
       <!-- ARM JOINTS (S1-S5) -->

Commit message: Fix S1/S3 servo direction, calibrate prismatic gripper, arm controller S1/S2/S3
ros2_control.xacro:
- Add direction=-1 to S1_joint and S3_joint: servos turned opposite to the
  URDF/RViz convention. Fixed in the driver (not the URDF axis) - the rad->tick
  write and tick->rad read are exact inverses, so motion and reported state flip
  together and RViz stays consistent.
- Map gripper_left_joint (servo 4) as a prismatic metres<->ticks joint, reusing
  the linear conversion (offset + value*ticks_per_rad). Calibrated on hardware:
  jaw CLOSED = tick 202 (0.0 m), OPEN = tick 437 (0.04 m) => offset=202,
  ticks_per_rad=5875 ticks/m, direction=1. Previously scaled as radians, so the
  joint read ~-0.49 (outside [0,0.04]) and the gripper MoveIt group could not plan.

jetank_controllers.yaml, controllers/arm_controller.yaml:
- arm_controller now actuates S1,S2,S3 only. S5 (servo 5) is the camera joint,
  intentionally left out of MoveIt; it remains a torque-held hardware interface.

Co-Authored-By: Claude Opus 4.8 (1M context) <noreply@anthropic.com>
Claude-Session: https://claude.ai/code/session_01DMTxWKRBqTNjSkyXQjoEtu

File: config/ros2_control.xacro (robot description, xacro)
@@ -49,4 +49,10 @@
         <state_interface name="velocity"/>
         <param name="servo_id">1</param>
+        <!-- Servo 1 turns opposite to the URDF/RViz convention. Invert in the
+             driver (NOT the URDF <axis>): the driver ignores URDF axis, and its
+             rad->tick write and tick->rad read are exact inverses, so flipping
+             direction reverses both commanded motion and reported state together,
+             keeping RViz consistent. Verified 2026-06-28 (arm-model audit). -->
+        <param name="direction">-1</param>
       </joint>
       <joint name="S2_joint">
@@ -67,4 +73,7 @@
         <state_interface name="velocity"/>
         <param name="servo_id">3</param>
+        <!-- Servo 3 turns opposite to URDF/RViz; invert in the driver (see
+             S1_joint note above). Verified 2026-06-28 (arm-model audit). -->
+        <param name="direction">-1</param>
       </joint>
       <!-- S4_joint disabled - Servo 4 controls gripper instead -->
@@ -119,4 +128,17 @@
         <state_interface name="velocity"/>
         <param name="servo_id">4</param>
+        <!-- PRISMATIC gripper jaw [0, 0.04 m]. The driver's generic linear map
+             ticks = offset + value*ticks_per_rad is reused here as METRES->ticks:
+               offset        = servo-4 tick at jaw CLOSED (value = 0.0 m)
+               ticks_per_rad = ticks per METRE = (open_tick - closed_tick) / 0.04
+               direction     = +1 (set -1 if OPENING the jaw DECREASES the tick)
+             CALIBRATED on hardware 2026-06-28: jaw fully CLOSED = servo-4 tick 202
+             (-> 0.0 m), fully OPEN = tick 437 (-> 0.04 m). So offset=202,
+             ticks_per_rad = (437-202)/0.04 = 5875 ticks/m, direction=+1 (tick rises
+             as the jaw opens). (Before this the value was scaled as radians, state
+             read ~-0.49 outside [0,0.04], and the gripper MoveIt group could not plan.) -->
+        <param name="offset">202</param>
+        <param name="ticks_per_rad">5875</param>
+        <param name="direction">1</param>
       </joint>
       <!-- gripper_right_joint: own command interface so Gazebo can physically
